File: 1_Hardware/PCB/LizardBot1_ControlBoard_v1/LizardBot1_ControlBoard_v1.kicad_pcb (KiCad board)
At the start: 4 copper layers, 147 parts, among them J201 XT60-M, J202 Receptable-P5.08-2P, J203 JST-PH-2-Male, J204 JST-PH-2-Male, J205 Receptable-P5.08-4P, J206 JST-PH-2-Male, J207 USB_C_Receptacle_PowerOnly_6P, J301 2.54mm (F), J302 2.54mm (F), J303 USB_C_Receptacle_USB2.0_16P, J401 JST-PH-6-Male, J402 JST-PH-6-Male, J501 JST-PH-3-Male, J502 JST-PH-2-Male, J601 2.54mm (F), J602 2.54mm (F), J603 2.54mm (F), Q201 SQ4425EY, Q301 UMH3N, Q501 AO3400A, Q502 BSS138, Q503 BSS138, Q504 AO3400A, SW201 SW_SPDT, SW301 SW_Push, SW302 SW_Push, SW303 SW_SPST, SW501 SW_Push, U201 MP2225, U202 AP2112K-3.3, U301 ESP32-WROOM-32E, U302 USBLC6-2P6, U303 CP2102N-Axx-xQFN24, U401 DRV8874, U402 DRV8874, U501 MIC5225, U502 ICM-20948

Commit message: Finished PCB routing. Updated ESP32 GPIO layout.
Parts:
- removed H105, H106: MountingHole_Pad, MountingHole:MountingHole_3.2mm_M3_Pad_Via
- removed the J204 at (-29.7, 38.8)
- removed J206: JST-PH-2-Male, Connector_JST:JST_PH_S2B-PH-K_1x02_P2.00mm_Horizontal
- removed SW303: SW_SPST, Button_Switch_THT:SW_Slide_SPDT_Straight_CK_OS102011MS2Q
- added FID101: Fiducial, Fiducial:Fiducial_1mm_Mask2mm, F.Cu at (99.0, 69.5)
- added FID102: Fiducial, Fiducial:Fiducial_1mm_Mask2mm, F.Cu at (99.0, 140.5)
- added FID103: Fiducial, Fiducial:Fiducial_1mm_Mask2mm, F.Cu at (225.0, 140.5)
- F201: footprint Fuse:Fuseholder_Clip-5x20mm_Littelfuse_519_Inline_P20.60x5.00mm_D1.00mm_Horizontal -> Project_FootprintLib:Fuseholder_LittelFuse_5x20mm_0PTF0078P
- J203: value JST-PH-2-Male -> Conn_02x03_Odd_Even; footprint Connector_JST:JST_PH_S2B-PH-K_1x02_P2.00mm_Horizontal -> Connector_PinHeader_2.54mm:PinHeader_2x03_P2.54mm_Vertical
- moved C308 300.2 mm to (179.2, 129.2)
- moved C306 298.0 mm to (174.5, 136.0), turned to -90 degrees
- moved R407 297.4 mm to (180.2, 83.8), turned to -90 degrees
- moved R408 295.3 mm to (178.0, 83.8), turned to 90 degrees
- moved C307 295.2 mm to (172.2, 136.0), turned to -90 degrees
- moved SW302 288.0 mm to (174.8, 122.0)
- moved J204 285.0 mm to (216.5, 116.4), turned to 90 degrees
- moved R305 284.4 mm to (176.5, 144.8), turned to -90 degrees
- moved R307 283.7 mm to (179.2, 135.5)
- moved R308 282.3 mm to (179.2, 137.5)
- moved R309 280.7 mm to (179.2, 133.5)
- moved R310 279.7 mm to (179.2, 131.5), turned to 180 degrees
- moved C405 279.4 mm to (170.5, 76.2)
- moved R406 278.9 mm to (160.8, 68.5), turned to 90 degrees
- moved C304 278.1 mm to (151.5, 139.8)
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- renumbered J205 to J204, J207 to J205
Connections:
- J201 pad 1: +BATT -> GND
- J201 pad 2: GND -> +BATT
- J301 pad 1: /MCU/MCU_BAT_STATUS -> /MCU/MCU_IO12_RES
- J301 pad 10: /MCU/MCU_BUZZER -> /MCU/ENC1_B
- J301 pad 2: /MCU/DRV1_IPROPI -> /MCU/MCU_IO2_LED
- J301 pad 3: /MCU/DRV1_nFAULT -> /MCU/MCU_IO0
- J301 pad 4: /MCU/ENC1_A -> /MCU/DRV1_nFAULT
- J301 pad 5: /MCU/ENC1_B -> /MCU/DRV1_nSLEEP
- J301 pad 6: /MCU/DRV2_IPROPI -> /MCU/DRV1_PH_IN2
- J301 pad 7: /MCU/DRV2_nFAULT -> /MCU/MCU_FAN_PWM
- J301 pad 8: /MCU/ENC2_A -> /MCU/DRV1_EN_IN1
- J301 pad 9: /MCU/ENC2_B -> /MCU/ENC1_A
- J302 pad 1: /MCU/DRV1_nSLEEP -> /MCU/MCU_BUZZER
- J302 pad 10: /MCU/MCU_IO12_RES -> /MCU/MCU_BAT_STATUS
- J302 pad 2: /MCU/DRV1_PH_IN2 -> /MCU/DRV2_EN_IN1
- J302 pad 3: /MCU/DRV1_EN_IN1 -> /MCU/DRV2_PH_IN2
- J302 pad 4: /MCU/MCU_FAN_PWM -> /MCU/DRV2_nSLEEP
- J302 pad 5: /MCU/DRV2_nSLEEP -> /MCU/DRV2_nFAULT
- J302 pad 6: /MCU/DRV2_PH_IN2 -> /MCU/ENC2_B
- J302 pad 7: /MCU/DRV2_EN_IN1 -> /MCU/ENC2_A
- J302 pad 8: /MCU/MCU_IO0 -> /MCU/DRV1_IPROPI
- J302 pad 9: /MCU/MCU_IO2_LED -> /MCU/DRV2_IPROPI
- J401 pad 1: /Motor_Driver/DRV1_OUT2 -> /Motor_Driver/DRV1_OUT1
- J401 pad 6: /Motor_Driver/DRV1_OUT1 -> /Motor_Driver/DRV1_OUT2
- J402 pad 1: /Motor_Driver/DRV2_OUT2 -> /Motor_Driver/DRV2_OUT1
- J402 pad 6: /Motor_Driver/DRV2_OUT1 -> /Motor_Driver/DRV2_OUT2
- SW201 pad 1: /Power_Supply/LDO_VIN -> +5V
- SW201 pad 2: Net-(D204-K) -> /Power_Supply/LDO_VIN
- SW201 pad 3: +5V -> Net-(D204-K)
- U301 pad 10: /MCU/DRV2_nFAULT -> /MCU/DRV2_nSLEEP
- U301 pad 11: /MCU/ENC2_A -> /MCU/DRV2_PH_IN2
- U301 pad 12: /MCU/ENC2_B -> /MCU/DRV2_EN_IN1
- U301 pad 26: /MCU/DRV2_EN_IN1 -> /MCU/DRV1_nFAULT
- U301 pad 27: /MCU/DRV2_PH_IN2 -> /MCU/DRV1_nSLEEP
- U301 pad 28: /MCU/DRV2_nSLEEP -> /MCU/DRV1_PH_IN2
- U301 pad 31: /MCU/DRV1_PH_IN2 -> /MCU/ENC1_A
- U301 pad 33: /MCU/DRV1_nSLEEP -> /MCU/ENC1_B
- U301 pad 5: /MCU/DRV1_IPROPI -> /MCU/DRV2_IPROPI
- U301 pad 6: /MCU/DRV1_nFAULT -> /MCU/DRV1_IPROPI
- U301 pad 7: /MCU/ENC1_A -> /MCU/ENC2_A
- U301 pad 8: /MCU/ENC1_B -> /MCU/ENC2_B
- U301 pad 9: /MCU/DRV2_IPROPI -> /MCU/DRV2_nFAULT
- U302 pad 1: /MCU/USBC_DN -> /MCU/USBC_DP
- U302 pad 3: /MCU/USBC_DP -> /MCU/USBC_DN
- U302 pad 4: /MCU/CP_DP -> /MCU/CP_USBC_DN
- U302 pad 6: /MCU/CP_DN -> /MCU/CP_USBC_DP
- U303 pad 3: /MCU/CP_DP -> /MCU/CP_USBC_DP
- U303 pad 4: /MCU/CP_DN -> /MCU/CP_USBC_DN
- U401 pad 3: /MCU/DRV2_nSLEEP -> /MCU/DRV1_nSLEEP
- U402 pad 3: /MCU/DRV1_nSLEEP -> /MCU/DRV2_nSLEEP
Routing:
- net +5V: track 0.00 -> 168.1 mm, vias 0 -> 4
- net /Communication_Interfaces/MCU_SDA: track 0.00 -> 151.6 mm, vias 0 -> 1
- net /Communication_Interfaces/MCU_SCL: track 0.00 -> 146.7 mm, vias 0 -> 2
- net /MCU/ENC1_B: track 0.00 -> 128.3 mm, vias 0 -> 1
- net /MCU/ENC1_A: track 0.00 -> 121.9 mm, vias 0 -> 1
- net /MCU/ENC2_A: track 0.00 -> 117.5 mm, vias 0 -> 1
- net /MCU/ENC2_B: track 0.00 -> 111.0 mm, vias 0 -> 1
- net GND: track 0.00 -> 110.9 mm, vias 0 -> 88
- net +3V3: track 0.00 -> 106.4 mm, vias 0 -> 13
- net /MCU/DRV1_EN_IN1: track 0.00 -> 99.4 mm
- net /MCU/DRV1_nFAULT: track 0.00 -> 98.2 mm, vias 0 -> 2
- net /MCU/DRV1_PH_IN2: track 0.00 -> 93.9 mm
- net /MCU/DRV1_nSLEEP: track 0.00 -> 93.0 mm
- net /MCU/DRV2_IPROPI: track 0.00 -> 83.7 mm, vias 0 -> 2
- net /MCU/DRV2_nFAULT: track 0.00 -> 80.4 mm, vias 0 -> 2
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- added copper zone on F.Cu, net +12V
- added copper zone on In2.Cu, net +12V
- added copper zone on In2.Cu, net +3V3
- added copper zone on In2.Cu, net +5V
- added copper zone on In2.Cu, net +BATT
- added copper zone on F.Cu, net /Power_Supply/BUCK_5V
- added copper zone on F.Cu, net /Power_Supply/BUCK_SW
- added copper zone on F.Cu, net /Power_Supply/E_SWITCH
- added copper zone on In2.Cu, net /Power_Supply/E_SWITCH
- added copper zone on In2.Cu, net /Power_Supply/M_SWITCH
- added copper zone on F.Cu, net GND
- added copper zone on In1.Cu, net GND
- added copper zone on In2.Cu, net Net-(J204-Pin_2)
Other:
- board outline added: 130 x 90 mm
