File: 1_Hardware/PCB/LizardBot1_ControlBoard_v1/Motor_Driver.kicad_sch (KiCad schematic)
At the start: 0 parts

Commit message: Added Motor_Driver schematic.
Parts:
- added C401, C405: 220uF, symbol Device:C_Polarized_Small_US
- added C402, C403, C406, C407: 0.1uF, symbol Device:C_Small
- added C404, C408: 22nF, symbol Device:C_Small
- added J401, J402: JST-PH-6-F, symbol Connector_Generic:Conn_01x06
- added JP401: PMODE as PWM, symbol Jumper:Jumper_2_Open
- added JP402: PMODE as PH/EN, symbol Jumper:Jumper_2_Open
- added JP403: IMODE as Level 3, symbol Jumper:Jumper_2_Open
- added JP404: IMODE as Level 2, symbol Jumper:Jumper_2_Open
- added JP405: IMODE as Level 1, symbol Jumper:Jumper_2_Open
- added R401: 62k, symbol Device:R_Small
- added R402: 20k, symbol Device:R_Small
- added R403, R407: 10k, symbol Device:R_Small
- added R404, R408: 1.2k, symbol Device:R_Small
- added R405: 16k, symbol Device:R_Small
- added R406: 50k, symbol Device:R_Small
- added U401, U402: ~, Package_SO:HTSSOP-16-1EP_4.4x5mm_P0.65mm_EP3.4x5mm_Mask3x3mm_ThermalVias, symbol Project_SymbolLib:DRV8874
Connections:
- new net: JP404.1 (A), R402.1
- new net: JP403.1 (A), R401.1
- new net +12V: C401.1, C402.1, C403.1, C405.1, C406.1, C407.1, U401.11 (VM), U402.11 (VM)
- new net +3V3: J401.2 (Pin_2), J402.2 (Pin_2), JP401.1 (A), R403.1, R405.1, R407.1
- new net DRV1_CPH: C404.2, U401.13 (CPH)
- new net DRV1_CPL: C404.1, U401.14 (CPL)
- new net DRV1_EN_IN1: U401.1 (EN/IN1)
- new net DRV1_IPROPI: R404.1, U401.6 (IPROPI)
- new net DRV1_OUT1: J401.6 (Pin_6), U401.8 (OUT1)
- new net DRV1_OUT2: J401.1 (Pin_1), U401.10 (OUT2)
- new net DRV1_PH_IN2: U401.2 (PH/IN2)
- new net DRV1_VCP: C403.2, U401.12 (VCP)
- new net DRV1_nFAULT: R403.2, U401.4 (~{nFAULT})
- new net DRV1_nSLEEP: U401.3 (~{nSLEEP})
- new net DRV2_CPH: C408.2, U402.13 (CPH)
- new net DRV2_CPL: C408.1, U402.14 (CPL)
- new net DRV2_EN_IN1: U402.1 (EN/IN1)
- new net DRV2_IPROPI: R408.1, U402.6 (IPROPI)
- new net DRV2_OUT1: J402.6 (Pin_6), U402.8 (OUT1)
- new net DRV2_OUT2: J402.1 (Pin_1), U402.10 (OUT2)
- new net DRV2_PH_IN2: U402.2 (PH/IN2)
- new net DRV2_VCP: C407.2, U402.12 (VCP)
- new net DRV2_nFAULT: R407.2, U402.4 (~{nFAULT})
- new net DRV2_nSLEEP: U402.3 (~{nSLEEP})
- new net DRV_IMODE: JP403.2 (B), JP404.2 (B), JP405.2 (B), U401.7 (IMODE), U402.7 (IMODE)
- new net DRV_PMODE: JP401.2 (B), JP402.2 (B), U401.16 (PMODE), U402.16 (PMODE)
- new net DRV_VREF: R405.2, R406.1, U401.5 (VREF), U402.5 (VREF)
- new net ENC1_A: J401.4 (Pin_4)
- new net ENC1_B: J401.3 (Pin_3)
- new net ENC2_A: J402.4 (Pin_4)
- new net ENC2_B: J402.3 (Pin_3)
- new net GND: C401.2, C402.2, C405.2, C406.2, J401.5 (Pin_5), J402.5 (Pin_5), JP402.1 (A), JP405.1 (A), R401.2, R402.2, R404.2, R406.2, R408.2, U401.15 (GND), U401.17 (PAD), U401.9 (PGND), U402.15 (GND), U402.17 (PAD), U402.9 (PGND)
Other:
- note added: "Auxiliary Driver Signals"
- note added: "IMODE Selector"
- note added: "IMODE State | nFAULT Response Quad-Level 1 = Fixed Off-Time (auto retry) Quad-Level 2 = Cycle-By-Cycle (auto retry) Quad-Level 3 = Cycle-By-Cycle (latched off) Quad-Level 4 (Hi-Z) = Fixed Off-Time (latched off)"
- note added: "I_TRIP = ±4.58A * V_REF = 2.5V * R_IPROPI = 1.2k * A_IPROPI = 455uA/A"
- note added: "Motor Connectors"
- note added: "Motor Driver Circuit"
- note added: "PMODE Selector"
- note added: "PMODE State | Control Mode Logic Low = PH/EN Logic High = PWM Hi-Z = Independent Half-Bridge"
- note added: "Voltage Reference"
- note added: "Voltage reference to set V_IPROPI and current regulation limit * set to 2.5V * if V_IPROPI == V_REF: current is limited"

Commit message: Added Peripherals schematic
Parts:
- U401, U402: value ~ -> DRV8874
Changed lines of the file:
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@@
 			)
 		)
-		(property "Value" "~"
-			(at 86.36 38.1 0)
+		(property "Value" "DRV8874"
+			(at 86.36 41.91 0)
 			(effects
 				(font
@@
 			)
 		)
-		(property "Value" "~"
-			(at 215.9 38.1 0)
-			(effects
-				(font
+		(property "Value" "DRV8874"
+			(at 215.9 41.91 0)
+			(effects
+				(font

Commit message: Added Communication_Interfaces schematic
Parts:
- J401, J402: value JST-PH-6-F -> JST-PH-6-Male
Changed lines of the file:
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@@
 		(dnp no)
 		(property "Reference" "J402"
-			(at 259.08 137.16 0)
-			(effects
-				(font
-					(size 1.27 1.27)
-				)
-				(justify left)
-			)
-		)
-		(property "Value" "JST-PH-6-F"
-			(at 259.08 154.94 0)
-			(effects
-				(font
-					(size 1.27 1.27)
-				)
-				(justify left)
+			(at 260.35 154.94 0)
+			(effects
+				(font
+					(size 1.27 1.27)
+				)
+			)
+		)
+		(property "Value" "JST-PH-6-Male"
+			(at 260.35 157.48 0)
+			(effects
+				(font
+					(size 1.27 1.27)
+				)
 			)
 		)
@@
 		(dnp no)
 		(property "Reference" "J401"
-			(at 259.08 106.68 0)
-			(effects
-				(font
-					(size 1.27 1.27)
-				)
-				(justify left)
-			)
-		)
-		(property "Value" "JST-PH-6-F"
-			(at 259.08 124.46 0)
-			(effects
-				(font
-					(size 1.27 1.27)
-				)
-				(justify left)
-			)
-		)
+			(at 260.35 124.46 0)
+			(effects
+				(font
+					(size 1.27 1.27)
+				)
+			)
+		)
+		(property "Value" "JST-PH-6-Male"
+			(at 260.35 127 0)
+			(effects
+				(font
+					(size 1.27 1.27)
+				)
+			)
+		)

Commit message: PCB schematics revision
Other:
- moved on the sheet: R403, R404, R407, R408

Commit message: Updated schematics. Assigned footprints. Added BOM to /4_Docs.
Parts:
- C401, C405: footprint (none) -> Capacitor_SMD:CP_Elec_8x10
- C402, C403, C406, C407: footprint (none) -> Capacitor_SMD:C_0603_1608Metric_Pad1.08x0.95mm_HandSolder
- C404, C408: footprint (none) -> Capacitor_SMD:C_0805_2012Metric_Pad1.18x1.45mm_HandSolder
- J401, J402: footprint (none) -> Connector_JST:JST_PH_S6B-PH-K_1x06_P2.00mm_Horizontal
- JP401, JP402, JP403, JP404, JP405: footprint (none) -> Jumper:SolderJumper-2_P1.3mm_Open_TrianglePad1.0x1.5mm
- R401, R402, R403, R404, R405, R406, R407, R408: footprint (none) -> Resistor_SMD:R_0805_2012Metric_Pad1.20x1.40mm_HandSolder
Changed lines of the file:
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@@
 			)
 		)
-		(property "Footprint" ""
+		(property "Footprint" "Resistor_SMD:R_0805_2012Metric_Pad1.20x1.40mm_HandSolder"
 			(at 127 46.99 0)
 			(effects
@@
 			)
 		)
-		(property "Footprint" ""
+		(property "Footprint" "Capacitor_SMD:CP_Elec_8x10"
 			(at 25.4 52.07 0)
 			(effects
@@
 			)
 		)
-		(property "Footprint" ""
+		(property "Footprint" "Jumper:SolderJumper-2_P1.3mm_Open_TrianglePad1.0x1.5mm"
 			(at 43.18 121.92 0)
 			(effects
@@
 			)
 		)
-		(property "Footprint" ""
+		(property "Footprint" "Resistor_SMD:R_0805_2012Metric_Pad1.20x1.40mm_HandSolder"
 			(at 182.88 135.89 0)
 			(effects
@@
 			)
 		)
-		(property "Footprint" ""
+		(property "Footprint" "Connector_JST:JST_PH_S6B-PH-K_1x06_P2.00mm_Horizontal"
 			(at 260.35 144.78 0)
 			(effects
@@
 			)
 		)
-		(property "Footprint" ""
+		(property "Footprint" "Resistor_SMD:R_0805_2012Metric_Pad1.20x1.40mm_HandSolder"
 			(at 99.06 133.35 0)
 			(effects
@@
 			)
 		)
-		(property "Footprint" ""
+		(property "Footprint" "Resistor_SMD:R_0805_2012Metric_Pad1.20x1.40mm_HandSolder"
 			(at 257.81 60.96 0)
 			(effects
@@
 			)
 		)
-		(property "Footprint" ""
+		(property "Footprint" "Resistor_SMD:R_0805_2012Metric_Pad1.20x1.40mm_HandSolder"
 			(at 128.27 60.96 0)
 			(effects
@@
 			)
 		)
-		(property "Footprint" ""
+		(property "Footprint" "Capacitor_SMD:C_0603_1608Metric_Pad1.08x0.95mm_HandSolder"
 			(at 166.37 52.07 0)
 			(effects
@@
 			)
 		)
-		(property "Footprint" ""
+		(property "Footprint" "Jumper:SolderJumper-2_P1.3mm_Open_TrianglePad1.0x1.5mm"
 			(at 116.84 138.43 0)
 			(effects
@@
 			)
 		)
-		(property "Footprint" ""
+		(property "Footprint" "Resistor_SMD:R_0805_2012Metric_Pad1.20x1.40mm_HandSolder"
 			(at 182.88 123.19 0)
 			(effects
@@
 			)
 		)
-		(property "Footprint" ""
+		(property "Footprint" "Capacitor_SMD:C_0603_1608Metric_Pad1.08x0.95mm_HandSolder"
 			(at 36.83 52.07 0)
 			(effects
@@
 			)
 		)
-		(property "Footprint" ""
+		(property "Footprint" "Capacitor_SMD:CP_Elec_8x10"
 			(at 154.94 52.07 0)
 			(effects
@@
 			)
 		)
-		(property "Footprint" ""
+		(property "Footprint" "Resistor_SMD:R_0805_2012Metric_Pad1.20x1.40mm_HandSolder"
 			(at 256.54 46.99 0)
 			(effects
@@
 			)
 		)
-		(property "Footprint" ""
+		(property "Footprint" "Capacitor_SMD:C_0805_2012Metric_Pad1.18x1.45mm_HandSolder"
 			(at 118.11 63.5 0)
 			(effects
@@
 			)
 		)
-		(property "Footprint" ""
+		(property "Footprint" "Resistor_SMD:R_0805_2012Metric_Pad1.20x1.40mm_HandSolder"
 			(at 93.98 123.19 0)
 			(effects
@@
 			)
 		)
-		(property "Footprint" ""
+		(property "Footprint" "Jumper:SolderJumper-2_P1.3mm_Open_TrianglePad1.0x1.5mm"
 			(at 43.18 132.08 0)
 			(effects
@@
 			)
 		)
-		(property "Footprint" ""
+		(property "Footprint" "Jumper:SolderJumper-2_P1.3mm_Open_TrianglePad1.0x1.5mm"
 			(at 116.84 128.27 0)
 			(effects
@@
 			)
 		)
-		(property "Footprint" ""
+		(property "Footprint" "Connector_JST:JST_PH_S6B-PH-K_1x06_P2.00mm_Horizontal"
 			(at 260.35 114.3 0)
 			(effects
@@
 			)
 		)
-		(property "Footprint" ""
+		(property "Footprint" "Capacitor_SMD:C_0603_1608Metric_Pad1.08x0.95mm_HandSolder"
 			(at 49.53 48.26 0)
 			(effects
@@
 			)
 		)
-		(property "Footprint" ""
+		(property "Footprint" "Jumper:SolderJumper-2_P1.3mm_Open_TrianglePad1.0x1.5mm"
 			(at 116.84 118.11 0)
 			(effects
@@
 			)
 		)
-		(property "Footprint" ""
+		(property "Footprint" "Capacitor_SMD:C_0805_2012Metric_Pad1.18x1.45mm_HandSolder"
 			(at 247.65 63.5 0)
 			(effects
@@
 			)
 		)
-		(property "Footprint" ""
+		(property "Footprint" "Capacitor_SMD:C_0603_1608Metric_Pad1.08x0.95mm_HandSolder"
 			(at 179.07 48.26 0)
 			(effects

Commit message: Finished PCB routing. Updated ESP32 GPIO layout.
Parts:
- JP401, JP402, JP403, JP404, JP405: now left out of the parts list
Connections:
- net DRV1_OUT1: now also J401.1 (Pin_1); no longer J401.6 (Pin_6)
- net DRV1_OUT2: now also J401.6 (Pin_6); no longer J401.1 (Pin_1)
- net DRV2_OUT1: now also J402.1 (Pin_1); no longer J402.6 (Pin_6)
- net DRV2_OUT2: now also J402.6 (Pin_6); no longer J402.1 (Pin_1)
Changed lines of the file:
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@@
 	(wire
 		(pts
+			(xy 55.88 60.96) (xy 71.12 60.96)
+		)
+		(stroke
+			(width 0)
+			(type default)
+		)
+	)
+	(wire
+		(pts
 			(xy 231.14 48.26) (xy 243.84 48.26)
 		)
@@
 	(wire
 		(pts
-			(xy 238.76 139.7) (xy 255.27 139.7)
-		)
-		(stroke
-			(width 0)
-			(type default)
-		)
-	)
-	(wire
-		(pts
 			(xy 128.27 55.88) (xy 143.51 55.88)
 		)
@@
 	(wire
 		(pts
-			(xy 231.14 60.96) (xy 252.73 60.96)
+			(xy 238.76 139.7) (xy 255.27 139.7)
 		)
 		(stroke
@@
 	(wire
 		(pts
-			(xy 127 49.53) (xy 127 53.34)
+			(xy 231.14 60.96) (xy 252.73 60.96)
 		)
 		(stroke
@@
 	(wire
 		(pts
-			(xy 121.92 128.27) (xy 128.27 128.27)
+			(xy 127 49.53) (xy 127 53.34)
 		)
 		(stroke
@@
 	(wire
 		(pts
-			(xy 101.6 45.72) (xy 114.3 45.72)
+			(xy 121.92 128.27) (xy 128.27 128.27)
 		)
 		(stroke
@@
 	(wire
 		(pts
-			(xy 86.36 181.61) (xy 105.41 181.61)
+			(xy 101.6 45.72) (xy 114.3 45.72)
 		)
 		(stroke
@@
 	(wire
 		(pts
-			(xy 238.76 109.22) (xy 255.27 109.22)
+			(xy 86.36 181.61) (xy 105.41 181.61)
 		)
 		(stroke
@@
 	(wire
 		(pts
-			(xy 55.88 60.96) (xy 71.12 60.96)
+			(xy 54.61 121.92) (xy 54.61 132.08)
 		)
 		(stroke
@@
 	(wire
 		(pts
-			(xy 54.61 121.92) (xy 54.61 132.08)
+			(xy 182.88 138.43) (xy 182.88 140.97)
 		)
 		(stroke
@@
 	(wire
 		(pts
-			(xy 182.88 138.43) (xy 182.88 140.97)
+			(xy 238.76 109.22) (xy 255.27 109.22)
 		)
 		(stroke
@@
 	)
 	(label "DRV2_OUT2"
+		(at 238.76 152.4 0)
+		(fields_autoplaced yes)
+		(effects
+			(font
+				(size 1.27 1.27)
+			)
+			(justify left bottom)
+		)
+	)
+	(label "DRV2_OUT1"
 		(at 238.76 139.7 0)
 		(fields_autoplaced yes)
@@
 		)
 	)
-	(label "DRV1_OUT1"
-		(at 238.76 121.92 0)
-		(fields_autoplaced yes)
-		(effects
-			(font
-				(size 1.27 1.27)
-			)
-			(justify left bottom)
-		)
-	)
 	(label "DRV2_OUT2"
 		(at 243.84 48.26 180)
@@
 		)
 	)
-	(label "DRV2_OUT1"
-		(at 238.76 152.4 0)
-		(fields_autoplaced yes)
-		(effects
-			(font
-				(size 1.27 1.27)
-			)
-			(justify left bottom)
-		)
-	)
 	(label "DRV1_EN_IN1"
 		(at 55.88 55.88 0)
@@
 	)
 	(label "DRV1_OUT2"
-		(at 238.76 109.22 0)
+		(at 238.76 121.92 0)
 		(fields_autoplaced yes)
 		(effects
@@
 		)
 	)
+	(label "DRV1_OUT1"
+		(at 238.76 109.22 0)
+		(fields_autoplaced yes)
+		(effects
+			(font
+				(size 1.27 1.27)
+			)
+			(justify left bottom)
+		)
+	)
 	(label "DRV2_IPROPI"
 		(at 273.05 55.88 180)
@@
 		(unit 1)
 		(exclude_from_sim yes)
-		(in_bom yes)
+		(in_bom no)
 		(on_board yes)
 		(dnp no)
@@
 		(unit 1)
 		(exclude_from_sim yes)
-		(in_bom yes)
+		(in_bom no)
 		(on_board yes)
 		(dnp no)
@@
 		(unit 1)
 		(exclude_from_sim yes)
-		(in_bom yes)
+		(in_bom no)
 		(on_board yes)
 		(dnp no)
@@
 		(unit 1)
 		(exclude_from_sim yes)
-		(in_bom yes)
+		(in_bom no)
 		(on_board yes)
 		(dnp no)
@@
 		(unit 1)
 		(exclude_from_sim yes)
-		(in_bom yes)
+		(in_bom no)
 		(on_board yes)
 		(dnp no)
